File: BQ51013B_Wireless_RX_Test.kicad_pcb (KiCad board)
At the start: 2 copper layers, 26 parts, among them J1 Conn_01x05, J2 Conn_01x01, J3 Conn_01x01, U1 BQ51013BRHLR

Commit message: layout 85% done
Parts:
- moved C1 5.46 mm to (141.4, 93.0)
- moved D1 4.79 mm to (146.8, 95.4), turned to -90 degrees
- moved C13 3.75 mm to (140.4, 88.5), turned to 45 degrees
- moved R4 3.13 mm to (145.2, 95.4), turned to -90 degrees
- moved C4 2.56 mm to (150.7, 89.1)
- moved R3 2.43 mm to (148.5, 95.4), turned to 90 degrees
- moved C7 2.42 mm to (141.4, 91.4)
- moved C14 2.09 mm to (150.1, 81.4), turned to 180 degrees
- moved C3 1.88 mm to (150.1, 83.4), turned to 180 degrees
- moved R2 1.81 mm to (143.6, 95.8), turned to -90 degrees
- moved C6 1.41 mm to (150.7, 90.6)
- moved C5 1.36 mm to (150.7, 92.2)
- moved R1 1.31 mm to (150.7, 93.7), turned to 180 degrees
- moved R5 1.27 mm to (154.2, 86.8)
- moved C12 0.99 mm to (152.5, 86.9), turned to -90 degrees
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Connections:
- U1 pad 22: (no net) -> GND
- U1 pad 23: (no net) -> GND
- U1 pad 24: (no net) -> GND
- U1 pad 25: (no net) -> GND
- U1 pad 26: (no net) -> GND
- U1 pad 27: (no net) -> GND
- U1 pad 28: (no net) -> GND
- U1 pad 29: (no net) -> GND
Routing:
- net Net-(J3-Pin_1): track 0.00 -> 49.1 mm, vias 0 -> 2
- net Net-(U1-AC1): track 0.00 -> 29.2 mm, vias 0 -> 2
- net /VOUT: track 0.00 -> 24.1 mm, vias 0 -> 2
- net /RECT: track 0.00 -> 18.7 mm, vias 0 -> 3
- net GND: track 0.00 -> 15.8 mm, vias 0 -> 10
- net Net-(U1-TS/CTRL): track 0.00 -> 11.5 mm
- net Net-(J2-Pin_1): track 0.00 -> 7.21 mm
- net Net-(U1-RECT): track 0.00 -> 6.80 mm
- net /EN2: track 0.00 -> 6.56 mm
- net /~{CHG}: track 0.00 -> 6.25 mm
- net /EN1: track 0.00 -> 4.92 mm
- net Net-(U1-FOD): track 0.00 -> 4.44 mm
- net Net-(U1-COMM1): track 0.00 -> 4.36 mm
- net Net-(U1-ILIM): track 0.00 -> 3.91 mm
- net Net-(U1-CLAMP1): track 0.00 -> 3.79 mm
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- added copper zone on B.Cu, net GND
